Commit message: use KDL for inverse kinematics

File: kuka_kr5_support/urdf/kr5_arc_macro.xacro (robot description, xacro)
@@ -5,5 +5,5 @@
     <!-- base link -->
     <link name="${prefix}base_link">
-      <inertial>
+      <!-- <inertial>
         <origin xyz="-0.017519394031846 8.11394768450848E-07 0.0975924044854325"
                 rpy="0 0 0" />
@@ -16,5 +16,5 @@
             iyz="-4.8990117845347E-07"
             izz="0.0514875586171667" />
-      </inertial>
+      </inertial> -->
       <visual>
         <origin rpy="0 0 0" xyz="0 0 0"/>
